File: KiCad/Keyboard.kicad_sch (KiCad schematic)
At the start: 69 parts, among them J1 USB_C_Receptacle, SW1 SW_Push, SW10 SW_Push, SW13 SW_Push, SW14 SW_Push, SW15 SW_Push, SW16 SW_Push, SW19 SW_Push, SW2 SW_Push, SW20 SW_Push, SW21 SW_Push, SW22 SW_Push, SW25 SW_Push, SW26 SW_Push, SW27 SW_Push, SW29 SW_Push, SW3 SW_Push, SW30 SW_Push, SW31 SW_Push, SW32 SW_Push, SW33 SW_Push, SW34 SW_Push, SW35 SW_Push, SW36 SW_Push, SW39 SW_Push, SW4 SW_Push, SW5 SW_Push, SW7 SW_Push, SW8 SW_Push, SW9 SW_Push, U1 ESP32-C6-MINI-1, U2 USBLC6-2SC6

Commit message: Pin allocation fixes
Parts:
- added R4: 10k, symbol Device:R_Small
Connections:
- net +3.3V: now also R4.1
- net OLED_SDA: now also U1.29 (IO23); no longer U1.20 (IO15)
- net ROW_2: now also D14.1 (K)
- net at U1.23 (IO9): now also R4.2
- no-connect marks 14 -> 13
Other:
- moved on the sheet: D14, SW14
Changed lines of the file:
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@@
 	)
 	(junction
+		(at 91.44 76.2)
+		(diameter 0)
+		(color 0 0 0 0)
+	)
+	(junction
 		(at 78.74 101.6)
 		(diameter 0)
@@
 	)
 	(junction
-		(at 76.2 81.28)
+		(at 101.6 68.58)
 		(diameter 0)
 		(color 0 0 0 0)
 	)
 	(junction
-		(at 104.14 88.9)
+		(at 76.2 81.28)
 		(diameter 0)
 		(color 0 0 0 0)
 	)
 	(junction
-		(at 260.35 40.64)
+		(at 104.14 88.9)
 		(diameter 0)
 		(color 0 0 0 0)
 	)
 	(junction
-		(at 101.6 69.85)
+		(at 260.35 40.64)
 		(diameter 0)
 		(color 0 0 0 0)
@@
 	)
 	(no_connect
-		(at 111.76 172.72)
-	)
-	(no_connect
 		(at 247.65 40.64)
 	)
@@
 	)
 	(no_connect
-		(at 81.28 167.64)
+		(at 111.76 154.94)
 	)
 	(no_connect
@@
 	(wire
 		(pts
-			(xy 111.76 154.94) (xy 123.19 154.94)
+			(xy 101.6 25.4) (xy 101.6 43.18)
 		)
 		(stroke
@@
 	(wire
 		(pts
-			(xy 101.6 25.4) (xy 101.6 43.18)
+			(xy 78.74 50.8) (xy 91.44 50.8)
 		)
 		(stroke
@@
 	(wire
 		(pts
-			(xy 78.74 50.8) (xy 91.44 50.8)
+			(xy 66.04 88.9) (xy 78.74 88.9)
 		)
 		(stroke
@@
 	(wire
 		(pts
-			(xy 66.04 88.9) (xy 78.74 88.9)
+			(xy 76.2 25.4) (xy 76.2 43.18)
 		)
 		(stroke
@@
 	(wire
 		(pts
-			(xy 76.2 25.4) (xy 76.2 43.18)
+			(xy 111.76 162.56) (xy 123.19 162.56)
 		)
 		(stroke
@@
 	(wire
 		(pts
-			(xy 111.76 162.56) (xy 123.19 162.56)
+			(xy 91.44 76.2) (xy 104.14 76.2)
 		)
 		(stroke
@@
 	(wire
 		(pts
-			(xy 101.6 69.85) (xy 101.6 81.28)
-		)
-		(stroke
-			(width 0)
-			(type default)
-		)
-	)
-	(wire
-		(pts
 			(xy 41.91 146.05) (xy 38.1 146.05)
 		)
@@
 	(wire
 		(pts
-			(xy 101.6 55.88) (xy 101.6 69.85)
+			(xy 101.6 55.88) (xy 101.6 68.58)
 		)
 		(stroke
@@
 	(wire
 		(pts
+			(xy 63.5 167.64) (xy 68.58 167.64)
+		)
+		(stroke
+			(width 0)
+			(type default)
+		)
+	)
+	(wire
+		(pts
 			(xy 82.55 134.62) (xy 96.52 134.62)
 		)
@@
 	(wire
 		(pts
+			(xy 101.6 68.58) (xy 101.6 81.28)
+		)
+		(stroke
+			(width 0)
+			(type default)
+		)
+	)
+	(wire
+		(pts
 			(xy 76.2 93.98) (xy 76.2 114.3)
 		)
@@
 	(wire
 		(pts
+			(xy 111.76 172.72) (xy 123.19 172.72)
+		)
+		(stroke
+			(width 0)
+			(type default)
+		)
+	)
+	(wire
+		(pts
 			(xy 267.97 43.18) (xy 267.97 40.64)
 		)
@@
 	(wire
 		(pts
-			(xy 78.74 76.2) (xy 104.14 76.2)
+			(xy 78.74 76.2) (xy 91.44 76.2)
 		)
 		(stroke
@@
 	(wire
 		(pts
+			(xy 73.66 167.64) (xy 81.28 167.64)
+		)
+		(stroke
+			(width 0)
+			(type default)
+		)
+	)
+	(wire
+		(pts
 			(xy 50.8 146.05) (xy 46.99 146.05)
 		)
@@
 		)
 	)
+	(label "OLED_SDA"
+		(at 123.19 172.72 180)
+		(effects
+			(font
+				(size 1.27 1.27)
+			)
+			(justify right bottom)
+		)
+	)
 	(label "ROW_1"
 		(at 123.19 162.56 180)
@@
 		)
 	)
-	(label "OLED_SDA"
-		(at 123.19 154.94 180)
-		(effects
-			(font
-				(size 1.27 1.27)
-			)
-			(justify right bottom)
-		)
-	)
 	(label "COL_0"
 		(at 72.39 144.78 0)
@@
 	(symbol
 		(lib_id "Device:D")
-		(at 91.44 73.66 90)
+		(at 91.44 72.39 90)
 		(unit 1)
 		(body_style 1)
@@
 		(fields_autoplaced yes)
 		(property "Reference" "D14"
-			(at 93.98 72.3899 90)
+			(at 93.98 71.1199 90)
 			(show_name no)
 			(do_not_autoplace no)
@@
 		)
 		(property "Value" "D"
-			(at 93.98 74.9299 90)
+			(at 93.98 73.6599 90)
 			(show_name no)
 			(do_not_autoplace no)
@@
 		)
 		(property "Footprint" ""
-			(at 91.44 73.66 0)
+			(at 91.44 72.39 0)
 			(hide yes)
 			(show_name no)
@@
 		)
 		(property "Datasheet" ""
-			(at 91.44 73.66 0)
+			(at 91.44 72.39 0)
 			(hide yes)
 			(show_name no)
@@
 		)
 		(property "Description" "Diode"
-			(at 91.44 73.66 0)
+			(at 91.44 72.39 0)
 			(hide yes)
 			(show_name no)
@@
 		)
 		(property "Sim.Device" "D"
-			(at 91.44 73.66 0)
+			(at 91.44 72.39 0)
 			(hide yes)
 			(show_name no)
@@
 		)
 		(property "Sim.Pins" "1=K 2=A"
-			(at 91.44 73.66 0)
+			(at 91.44 72.39 0)
 			(hide yes)
 			(show_name no)
@@
 	)
 	(symbol
+		(lib_id "Device:R_Small")
+		(at 71.12 167.64 90)
+		(unit 1)
+		(body_style 1)
+		(exclude_from_sim no)
+		(in_bom yes)
+		(on_board yes)
+		(in_pos_files yes)
+		(dnp no)
+		(fields_autoplaced yes)
+		(property "Reference" "R4"
+			(at 71.12 162.56 90)
+			(show_name no)
+			(do_not_autoplace no)
+			(effects
+				(font
+					(size 1.016 1.016)
+				)
+			)
+		)
+		(property "Value" "10k"
+			(at 71.12 165.1 90)
+			(show_name no)
+			(do_not_autoplace no)
+			(effects
+				(font
+					(size 1.27 1.27)
+				)
+			)
+		)
+		(property "Footprint" ""
+			(at 71.12 167.64 0)
+			(hide yes)
+			(show_name no)
+			(do_not_autoplace no)
+			(effects
+				(font
+					(size 1.27 1.27)
+				)
+			)
+		)
+		(property "Datasheet" ""
+			(at 71.12 167.64 0)
+			(hide yes)
+			(show_name no)
+			(do_not_autoplace no)
+			(effects
+				(font
+					(size 1.27 1.27)
+				)
+			)
+		)
+		(property "Description" "Resistor, small symbol"
+			(at 71.12 167.64 0)
+			(hide yes)
+			(show_name no)
+			(do_not_autoplace no)
+			(effects
+				(font
+					(size 1.27 1.27)
+				)
+			)
+		)
+		(pin "1"
+		)
+		(pin "2"
+		)
+		(instances
+			(project "Keyboard"
+				(path "/8c50ca30-7e5f-4942-aa3e-2d9da8c7d0f2"
+					(reference "R4")
+					(unit 1)
+				)
+			)
+		)
+	)
+	(symbol
 		(lib_id "power:+5V")
 		(at 215.9 57.15 0)
@@
 	(symbol
 		(lib_id "Switch:SW_Push")
-		(at 96.52 69.85 0)
+		(at 96.52 68.58 0)
 		(unit 1)
 		(body_style 1)
@@
 		(fields_autoplaced yes)
 		(property "Reference" "SW14"
-			(at 96.52 62.23 0)
+			(at 96.52 60.96 0)
 			(show_name no)
 			(do_not_autoplace no)
@@
 		)
 		(property "Value" "SW_Push"
-			(at 96.52 64.77 0)
+			(at 96.52 63.5 0)
 			(show_name no)
 			(do_not_autoplace no)
@@
 		)
 		(property "Footprint" ""
-			(at 96.52 64.77 0)
+			(at 96.52 63.5 0)
 			(hide yes)
 			(show_name no)
@@
 		)
 		(property "Datasheet" ""
-			(at 96.52 64.77 0)
+			(at 96.52 63.5 0)
 			(hide yes)
 			(show_name no)
@@
 		)
 		(property "Description" "Push button switch, generic, two pins"
-			(at 96.52 69.85 0)
+			(at 96.52 68.58 0)
 			(hide yes)
 			(show_name no)
@@
 					(unit 1)
 				)
+			)
+		)
+	)
+	(symbol
+		(lib_id "power:+3.3V")
+		(at 63.5 167.64 90)
+		(unit 1)
+		(body_style 1)
+		(exclude_from_sim no)
+		(in_bom yes)
+		(on_board yes)
+		(in_pos_files yes)
+		(dnp no)
+		(fields_autoplaced yes)
+		(property "Reference" "#PWR017"
+			(at 67.31 167.64 0)
+			(hide yes)
+			(show_name no)
+			(do_not_autoplace no)
+			(effects
+				(font
+					(size 1.27 1.27)
+				)
+			)
+		)
+		(property "Value" "+3.3V"
+			(at 59.69 167.6399 90)
+			(show_name no)
+			(do_not_autoplace no)
+			(effects
+				(font
+					(size 1.27 1.27)
+				)
+				(justify left)
+			)
+		)
+		(property "Footprint" ""
+			(at 63.5 167.64 0)
+			(hide yes)
+			(show_name no)
+			(do_not_autoplace no)
+			(effects
+				(font
+					(size 1.27 1.27)
+				)
+			)
+		)
+		(property "Datasheet" ""
+			(at 63.5 167.64 0)
+			(hide yes)
+			(show_name no)
+			(do_not_autoplace no)
+			(effects
+				(font
+					(size 1.27 1.27)
+				)
+			)
+		)
+		(property "Description" "Power symbol creates a global label with name \"+3.3V\""
+			(at 63.5 167.64 0)
+			(hide yes)
+			(show_name no)
+			(do_not_autoplace no)
+			(effects
+				(font
+					(size 1.27 1.27)
+				)
+			)
+		)
+		(pin "1"
+		)
+		(instances
+			(project "Keyboard"
+				(path "/8c50ca30-7e5f-4942-aa3e-2d9da8c7d0f2"
+					(reference "#PWR017")
+					(unit 1)
+				)

Commit message: Mr. Krabs, I have an idea
Use SBU pins for one-way, orientation-independent UART RX
Connections:
- net RIGHT_RX: now reaches U1.30 (RXD0)
- net RIGHT_RX: now also J1.A8 (SBU1), J1.B8 (SBU2)
- no-connect marks 13 -> 12
Changed lines of the file:
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@@
+	)
+	(junction
+		(at 214.63 40.64)
+		(diameter 0)
+		(color 0 0 0 0)
 	)
 	(junction
@@
 	)
 	(no_connect
-		(at 217.17 40.64)
+		(at 111.76 139.7)
 	)
 	(no_connect
@@
 	)
 	(no_connect
-		(at 214.63 40.64)
-	)
-	(no_connect
 		(at 81.28 165.1)
 	)
@@
 	(wire
 		(pts
+			(xy 214.63 40.64) (xy 214.63 49.53)
+		)
+		(stroke
+			(width 0)
+			(type default)
+		)
+	)
+	(wire
+		(pts
 			(xy 33.02 24.13) (xy 38.1 24.13)
 		)
@@
 	(wire
 		(pts
+			(xy 111.76 142.24) (xy 123.19 142.24)
+		)
+		(stroke
+			(width 0)
+			(type default)
+		)
+	)
+	(wire
+		(pts
 			(xy 72.39 160.02) (xy 81.28 160.02)
 		)
@@
 		(pts
 			(xy 33.02 29.21) (xy 50.8 29.21)
+		)
+		(stroke
+			(width 0)
+			(type default)
+		)
+	)
+	(wire
+		(pts
+			(xy 214.63 40.64) (xy 217.17 40.64)
 		)
 		(stroke
@@
 		)
 	)
+	(label "RIGHT_RX"
+		(at 123.19 142.24 180)
+		(effects
+			(font
+				(size 1.27 1.27)
+			)
+			(justify right bottom)
+		)
+	)
 	(label "D-"
 		(at 260.35 53.34 90)
@@
 		)
 	)
+	(label "RIGHT_RX"
+		(at 214.63 49.53 90)
+		(effects
+			(font
+				(size 1.27 1.27)
+			)
+			(justify left bottom)
+		)
+	)
